File: NS ELRS RX MICRO.kicad_sch (KiCad schematic)
At the start: 2 parts, among them U1 ESP32-C3, U2 SX1280IMLTRT

Commit message: commit
Parts:
- added FL1: 2450FM07D0034, Filter:Filter_1109-5_1.1x0.9mm, symbol Filter:B39162B8813P810
- added U3: SE2431L-R, SE2431L_SKY, symbol 2026-10-20_12-47-49:SE2431L-R
Connections:
- new net: FL1.2, FL1.5
Other:
- moved on the sheet: U1, U2

Commit message: 80pct schematic drawn
Parts:
- added C1, C2: 10uF, Package_SON:WSON-6-1EP_2x2mm_P0.65mm_EP1x1.6mm_ThermalVias, symbol Device:C
- added C10, C13: 10nF, Package_SON:WSON-6-1EP_2x2mm_P0.65mm_EP1x1.6mm_ThermalVias, symbol Device:C
- added C11, C12, C4: 100nF, Package_SON:WSON-6-1EP_2x2mm_P0.65mm_EP1x1.6mm_ThermalVias, symbol Device:C
- added C14: 470nF, Package_SON:WSON-6-1EP_2x2mm_P0.65mm_EP1x1.6mm_ThermalVias, symbol Device:C
- added C3, C5: 10pF, Package_SON:WSON-6-1EP_2x2mm_P0.65mm_EP1x1.6mm_ThermalVias, symbol Device:C
- added C6, C7, C8, C9: 1.2pF, Package_SON:WSON-6-1EP_2x2mm_P0.65mm_EP1x1.6mm_ThermalVias, symbol Device:C
- added J1, J2: Conn_Coaxial, Package_SON:WSON-6-1EP_2x2mm_P0.65mm_EP1x1.6mm_ThermalVias, symbol Connector:Conn_Coaxial
- added L1, L2: 3nH, symbol Device:L
- added L3: 15uH, symbol Device:L
- added R1: 100k, symbol Device:R
- added R2: 2.2k, symbol Device:R
- added R3: 1.2k, symbol Device:R
- added U4: LP5912-3.3DRV, Package_SON:WSON-6-1EP_2x2mm_P0.65mm_EP1x1.6mm_ThermalVias, symbol Regulator_Linear:LP5912-3.3DRV
- added Y1: 52MHz, 8pF, Oscillator:Oscillator_SMD_SeikoEpson_SG210-4Pin_2.5x2.0mm, symbol Device:Crystal_GND24
Connections:
- net GND: now also FL1.2, FL1.4, FL1.5, U2.25 (EXP), U3.10 (GND), U3.11 (GND), U3.12 (GND), U3.14 (GND), U3.18 (GND), U3.25 (EPAD), U3.9 (GND), C1.2, C10.2, C11.1, C12.1, C13.1, C14.2, C2.2, C3.2, C4.2, C5.2, C6.2, C7.2, C8.2, C9.2, J1.2 (Ext), J2.2 (Ext), R1.1, U4.5 (GND), U4.7 (EP), Y1.2 (G), Y1.4 (G)
- net at U3.1 (B2): now also R2.2
- net ANT2: now reaches U3.13 (ANT2)
- net ANT2: now also C8.1, L2.1
- net ANT1: now reaches U3.15 (ANT1)
- net ANT1: now also C7.1, L1.1
- net ANT_SEL: now reaches U3.16 (ANT_SEL)
- net +3V3: now reaches U3.19 (VCC2)
- net +3V3: now also U3.20 (CSD), U3.21 (CPS), U3.22 (VCC1), C2.1, C3.1, C4.1, C5.1, U4.1 (OUT)
- net at U3.2 (B1): now also R3.2
- net BOUT: now reaches U3.23 (BOUT)
- net BOUT: now also R2.1, R3.1
- net PWR_TXEN: now reaches U3.24 (CTX)
- net PWR_TXEN: now also R1.2
- net FRONTEND_IN: now reaches U3.6 (T/R)
- net FRONTEND_IN: now also FL1.3
- net at U2.1 (VR_PA): now also C10.1
- net at U2.11 (VBAT_IO): now also C11.2
- net V_DCC: now reaches U2.12 (DCC_FB)
- net V_DCC: now also U2.2 (VDD_IN), C13.2, C14.1, L3.1
- net V_DCC2: now reaches U2.14 (DCC_SW)
- net V_DCC2: now also L3.2
- net at U2.15 (VBAT): now also C12.2
- net RADIO_OUT: now reaches U2.22 (RFIO)
- net RADIO_OUT: now also FL1.1
- net RST: now reaches U2.3 (~{RESET})
- net at U2.4 (XTA): now also Y1.1
- net at U2.6 (XTB): now also Y1.3
- net BUSY: now reaches U2.7 (BUSY)
- net DIO: now reaches U2.8 (DIO1)
- new net: C6.1, J1.1 (In), L1.2
- new net: C9.1, J2.1 (In), L2.2
- new net +5V: C1.1, U4.4 (EN), U4.6 (IN)
- no-connect marks 0 -> 3
Other:
- moved on the sheet: FL1, U1

Commit message: more updates!
Parts:
- added AE1: Antenna_Chip, Oscillator:Oscillator_SMD_SeikoEpson_SG210-4Pin_2.5x2.0mm, symbol Device:Antenna_Chip
- added C15: 10uF, Package_SON:WSON-6-1EP_2x2mm_P0.65mm_EP1x1.6mm_ThermalVias, symbol Device:C
- added C16, C19: 1uF, Package_SON:WSON-6-1EP_2x2mm_P0.65mm_EP1x1.6mm_ThermalVias, symbol Device:C
- added C17, C18: 0.1uF, Package_SON:WSON-6-1EP_2x2mm_P0.65mm_EP1x1.6mm_ThermalVias, symbol Device:C
- added C20, C21: 12pF, Package_SON:WSON-6-1EP_2x2mm_P0.65mm_EP1x1.6mm_ThermalVias, symbol Device:C
- added R4: 10k, symbol Device:R
- added R5: 0R, symbol Device:R
- added Y2: 40MHz, 8pF, Oscillator:Oscillator_SMD_SeikoEpson_SG210-4Pin_2.5x2.0mm, symbol Device:Crystal_GND24
Connections:
- net +3V3: now also U1.11 (VDD3P3_RTC), U1.17 (VDD3P3_CPU), U1.18 (VDD_SPI), U1.2 (VDD3P3), U1.3 (VDD3P3), U1.31 (VDDA), U1.32 (VDDA), C15.2, C16.2, C17.2, C18.2, R4.2
- net GND: now also U1.33 (GND), AE1.2 (PCB_Trace), C15.1, C16.1, C17.1, C18.1, C19.1, C20.1, C21.1, Y2.2 (G), Y2.4 (G)
- net MISO: now reaches U2.16 (MISO_TX)
- net MOSI: now reaches U2.17 (MOSI_RX)
- net SCK: now reaches U2.18 (SCK_~{RTS})
- net CS: now reaches U2.19 (~{SS_CTS})
- net at U1.1 (LNA_IN): now also R5.1
- net at U1.29 (XTAL_N): now also C20.2, Y2.1
- net at U1.30 (XTAL_P): now also C21.2, Y2.3
- net at U1.7 (CHIP_EN): now also C19.2, R4.1
- new net: AE1.1 (FEED), R5.2
Other:
- moved on the sheet: C3, C4, C5, C6, C7, C8, C9, FL1, J1, J2, L1, L2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

Commit message: completed schematic
Parts:
- removed U3: SE2431L-R, SE2431L_SKY, symbol 2026-10-20_12-47-49:SE2431L-R
- added C22: 1uF, Package_SON:WSON-6-1EP_2x2mm_P0.65mm_EP1x1.6mm_ThermalVias, symbol Device:C
- added D1: LED, symbol Device:LED
- added J10, J11: Conn_01x01_Female, TestPoint:TestPoint_Pad_1.0x1.0mm, symbol Connector:Conn_01x01_Female
- added J3, J4, J5, J6: Conn_01x01_Female, TestPoint:TestPoint_Pad_2.5x2.5mm, symbol Connector:Conn_01x01_Female
- added J7: Conn_01x04_Male, Connector_JST:JST_GH_SM04B-GHS-TB_1x04-1MP_P1.25mm_Horizontal, symbol Connector:Conn_01x04_Male
- added R6, R7: 10k, symbol Device:R
- added R8: 1k, symbol Device:R
- added R9: 10k, Resistor_SMD:R_0402_1005Metric, symbol Device:R
- added TP1: USBD-, Package_DIP:DIP-16_W7.62mm, symbol Connector:TestPoint
- added TP2: USBD+, Package_DIP:DIP-16_W7.62mm, symbol Connector:TestPoint
- added U6: SE2431L, Package_DFN_QFN:QFN-24-1EP_3x4mm_P0.4mm_EP1.65x2.65mm, symbol Anyleaf Shared:SE2431L
- AE1: footprint Oscillator:Oscillator_SMD_SeikoEpson_SG210-4Pin_2.5x2.0mm -> RF_Antenna:Johanson_2450AT18x100
- FL1: footprint Filter:Filter_1109-5_1.1x0.9mm -> 2450FM07D0034:2450FM07D0034
- J1, J2: footprint Package_SON:WSON-6-1EP_2x2mm_P0.65mm_EP1x1.6mm_ThermalVias -> Connector_Coaxial:U.FL_Hirose_U.FL-R-SMT-1_Vertical
- U4: footprint Package_SON:WSON-6-1EP_2x2mm_P0.65mm_EP1x1.6mm_ThermalVias -> Package_TO_SOT_SMD:TSOT-23-5
Connections:
- net +3V3: now also R6.1, R7.1, R8.1, R9.1, U6.19 (VCC2), U6.20 (CSD), U6.21 (CPS), U6.22 (VCC1); no longer U1.18 (VDD_SPI)
- net +5V: now also J4.1 (Pin_1), J7.3 (Pin_3)
- net ANT1: now also U6.15 (ANT1)
- net ANT2: now also U6.13 (ANT2)
- net ANT_SEL: now also U1.16 (GPIO10), U6.16 (ANT_SEL)
- net BOUT: now also U6.23 (BOUT)
- net BUSY: now also U1.8 (GPIO3)
- net CS: now also U1.13 (MTDO), R7.2
- net DIO: now also U1.5 (XTAL_32K_N)
- net FRONTEND_IN: now also U6.6 (TR)
- net GND: now also C22.2, J11.1 (Pin_1), J3.1 (Pin_1), J7.4 (Pin_4), U6.10 (GND), U6.11 (GND), U6.12 (GND), U6.14 (GND), U6.18 (GND), U6.25 (GND_EP), U6.9 (GND)
- net MISO: now also U1.10 (MTDI)
- net MOSI: now also U1.12 (MTCK)
- net PWR_TXEN: now also U1.4 (XTAL_32K_P), U6.24 (CTX)
- net RST: now also U1.6 (GPIO2), R6.2
- net SCK: now also U1.9 (MTMS)
- net at R2.2: now also U6.1 (B2)
- net at R3.2: now also U6.2 (B1)
- net ELRS_LED: now reaches U1.14 (GPIO8)
- net ELRS_LED: now also D1.1 (K)
- net at U1.15 (GPIO9): now also J10.1 (Pin_1), R9.2
- net at U1.25 (GPIO18): now also TP1.1
- net at U1.26 (GPIO19): now also TP2.1
- net RX: now reaches U1.27 (U0RXD)
- net RX: now also J6.1 (Pin_1), J7.1 (Pin_1)
- net TX: now reaches U1.28 (U0TXD)
- net TX: now also J5.1 (Pin_1), J7.2 (Pin_2)
- new net: D1.2 (A), R8.2
- new net VDD_SPI: C22.1, U1.18 (VDD_SPI)
- no-connect marks 3 -> 9
Other:
- note added: "JST GH Pin for FC"
- note added: "Pads for FC"
- moved on the sheet: C1, C2, C3, C4, C5, FL1, R1, R2, R3, U4

Commit message: completed pcb routing
Parts:
- removed U4: LP5912-3.3DRV, Package_TO_SOT_SMD:TSOT-23-5, symbol Regulator_Linear:LP5912-3.3DRV
- added U3: 3.3V, 500mA, Package_TO_SOT_SMD:TSOT-23-5, symbol water_monitor-rescue:MCP1802-3.3-Anyleaf_shared
- C1: value 10uF -> 1uF; footprint Package_SON:WSON-6-1EP_2x2mm_P0.65mm_EP1x1.6mm_ThermalVias -> Capacitor_SMD:C_0402_1005Metric; LCSC (none) -> C52923
- C10, C11, C12, C13, C14, C15, C16, C17, C18, C19, C20, C21, C22, C3, C4, C5, C6, C7, C8, C9: footprint Package_SON:WSON-6-1EP_2x2mm_P0.65mm_EP1x1.6mm_ThermalVias -> Capacitor_SMD:C_0402_1005Metric
- C2: value 10uF -> 2.2uF; footprint Package_SON:WSON-6-1EP_2x2mm_P0.65mm_EP1x1.6mm_ThermalVias -> Capacitor_SMD:C_0402_1005Metric; LCSC (none) -> C12530
- D1: footprint (none) -> LED_SMD:LED_0603_1608Metric
- L1, L2: footprint (none) -> Inductor_SMD:L_0402_1005Metric
- L3: footprint (none) -> Inductor_SMD:L_0805_2012Metric
- R1, R2, R3, R4, R6, R7: footprint (none) -> Resistor_SMD:R_0402_1005Metric
- R5, R8: footprint (none) -> Resistor_SMD:R_0201_0603Metric
- TP1, TP2: footprint Package_DIP:DIP-16_W7.62mm -> TestPoint:TestPoint_Pad_1.0x1.0mm
- Y1: footprint Oscillator:Oscillator_SMD_SeikoEpson_SG210-4Pin_2.5x2.0mm -> Crystal:Crystal_SMD_2016-4Pin_2.0x1.6mm
- Y2: footprint Oscillator:Oscillator_SMD_SeikoEpson_SG210-4Pin_2.5x2.0mm -> Crystal:Crystal_SMD_2520-4Pin_2.5x2.0mm
Connections:
- net +3V3: now also C11.2, C12.2, C2.2, U2.11 (VBAT_IO), U2.15 (VBAT), U3.5 (VOUT); no longer C2.1
- net GND: now also C1.1, C2.1, U3.2 (GND); no longer C1.2, C2.2
- net +5V renamed PWR_IN
- net PWR_IN: now also C1.2, U3.1 (VIN), U3.3 (~{SHDN}); no longer C1.1
- no-connect marks 9 -> 8
