File: NS ELRS RX MICRO.kicad_pcb (KiCad board)
At the start: 4 copper layers, 18.2 x 24.1 mm, 54 parts, among them J1 Conn_Coaxial, J10 Conn_01x01_Female, J11 Conn_01x01_Female, J2 Conn_Coaxial, J3 Conn_01x01_Female, J7 Conn_01x04_Male, U1 ESP32-C3, U2 SX1280IMLTRT, U3 3.3V, 500mA, U6 SE2431L, Y1 52MHz, 8pF, Y2 40MHz, 8pF

Commit message: fixed some errors
Parts:
- moved C13 0.33 mm to (170.1, 95.0)
- moved R1 0.20 mm to (171.2, 95.2)
- moved C18 0.16 mm to (175.4, 94.2)
Routing:
- net /V_DCC: track 6.39 -> 14.3 mm, vias 0 -> 2
- net +3V3: track 64.2 -> 70.7 mm
- net GND: track 44.0 -> 49.9 mm, vias 23 -> 46
- net /PWR_TXEN: track 14.1 -> 9.96 mm, vias 4 -> 3
- net /PWR_IN: track 10.7 -> 14.1 mm
- net /MOSI: track 16.7 -> 18.0 mm
- net /CS: track 17.0 -> 17.9 mm
